File: b_Regulador_tension_variable/b_Regulador_tension_variable.kicad_sch (KiCad schematic)
At the start: 10 parts, among them J1 Screw_Terminal_01x02, J2 Screw_Terminal_01x02, U1 LM317_TO-252

Commit message: .
Parts:
- C1: value C -> 0.1u; footprint (none) -> Capacitor_SMD:C_0201_0603Metric
- C2: value C_Polarized -> 1u; footprint (none) -> Capacitor_SMD:CP_Elec_6.3x5.8
- C3: value C_Polarized -> 10u; footprint (none) -> Capacitor_SMD:CP_Elec_6.3x5.8
- D1, D2: value D -> 1N4001; footprint (none) -> Diode_SMD:D_SMA
- J1, J2: footprint (none) -> TerminalBlock_Phoenix:TerminalBlock_Phoenix_MKDS-1,5-2_1x02_P5.00mm_Horizontal
- R1: value R -> 240; footprint (none) -> Resistor_SMD:R_1206_3216Metric
- RV1: value R_Potentiometer -> 5k
Connections:
- net GND: now also J2.1 (Pin_1); no longer J2.2 (Pin_2)
- net V_OUT: now reaches C2.1, D1.2 (A), D2.1 (K), R1.1, U1.2 (VO)
- net V_OUT: now also J2.2 (Pin_2); no longer J2.1 (Pin_1)
Other:
- moved on the sheet: D1, J1, J2
